Commit message: update from tamar

File: src/arm_robot_description/urdf/arm_description2.urdf.xacro (robot description, xacro)
@@ -4,21 +4,8 @@
     <!-- Properties -->
     <xacro:property name="link_radius" value="0.0125" />
-    <xacro:property name="joint_length" value="0.05" />
-    <xacro:property name="link1_length" value="0.10" />
-    <xacro:property name="link2_length" value="0.05" />
-    <xacro:property name="link3_length" value="0.04" />
+    <xacro:property name="link_length" value="0.1" />
     <xacro:property name="payload_radius" value="0.0125" />
     <!-- Base footprint and link -->
-    <link name="base_footprint">
-        <inertial>
-            <mass value="0.001"/>
-            <inertia ixx="0.001" ixy="0.0" ixz="0.0" iyy="0.001" iyz="0.0" izz="0.001"/>
-        </inertial>
-        <collision>
-            <geometry>
-                <box size="0.001 0.001 0.001"/>
-            </geometry>
-        </collision>
-    </link>
+    <link name="base_footprint"/>
     <joint name="base_joint" type="revolute">
         <parent link="base_footprint"/>
@@ -31,5 +18,5 @@
             <visual>
                 <geometry>
-                    <cylinder radius="${link_radius}" length="${joint_length}"/>
+                    <cylinder radius="${link_radius}" length="${link_length}"/>
                 </geometry>
                 <material name="black"/>
@@ -37,35 +24,36 @@
             <collision>
                 <geometry>
-                    <cylinder radius="${link_radius}" length="${joint_length}"/>
+                    <cylinder radius="${link_radius}" length="${link_length}"/>
                 </geometry>
             </collision>
-            <xacro:cylinder_inertia m="0.1" r="${link_radius}" h="${joint_length}"
+            <xacro:cylinder_inertia m="0.1" r="${link_radius}" h="${link_length}"
                                     xyz="0 0 0" rpy="0 0 0" />
         </link>
     <joint name="base_link2_joint" type="fixed">
         <parent link="base_link"/>
-        <child link="link1"/>
-        <origin xyz="0 ${link1_length/2} 0" rpy="${-pi/2} 0 0 "/>
+        <child link="link2"/>
+        <origin xyz="0 0 0" rpy="${-pi/2} 0 0 "/>
         <axis xyz="0 1 0"/>
     </joint>
-    <link name="link1">
+    <link name="link2">
             <visual>
                 <geometry>
-                    <cylinder radius="${link_radius}" length="${link1_length}"/>
+                    <cylinder radius="${link_radius}" length="${link_length}"/>
                 </geometry>
                 <material name="blue"/>
+                <origin xyz="0 0 ${link_length/2}" rpy="0 0 0 "/>
             </visual>
             <collision>
                 <geometry>
-                    <cylinder radius="${link_radius}" length="${link1_length}"/>
+                    <cylinder radius="${link_radius}" length="${link_length}"/>
                 </geometry>
             </collision>
-            <xacro:cylinder_inertia m="0.1" r="${link_radius}" h="${link1_length}"
+            <xacro:cylinder_inertia m="0.1" r="${link_radius}" h="${link_length}"
                                     xyz="0 0 0" rpy="0 0 0" />
     </link>
-    <joint name="link1_joint2" type="revolute">
-        <parent link="link1"/>
+    <joint name="link2_joint2" type="revolute">
+        <parent link="link2"/>
         <child link="joint2_link"/>
-        <origin xyz="0 0 ${link1_length/2}" rpy="${pi/2} 0 0"/>
+        <origin xyz="0 0 ${link_length}" rpy="${pi/2} 0 0"/>
         <limit effort="100.0" velocity="10.0" lower="${-pi/2}" upper="${pi/2}" />
         <axis xyz="0 0 1"/>
@@ -74,41 +62,43 @@
             <visual>
                 <geometry>
-                    <cylinder radius="${link_radius}" length="${joint_length}"/>
+                    <cylinder radius="${link_radius}" length="${link_length}"/>
                 </geometry>
                 <material name="black"/>
+                <origin xyz="0 0 0" rpy="0 0 0"/>
             </visual>
             <collision>
                 <geometry>
-                    <cylinder radius="${link_radius}" length="${joint_length}"/>
+                    <cylinder radius="${link_radius}" length="${link_length}"/>
                 </geometry>
             </collision>
-            <xacro:cylinder_inertia m="0.1" r="${link_radius}" h="${joint_length}"
+            <xacro:cylinder_inertia m="0.1" r="${link_radius}" h="${link_length}"
                                     xyz="0 0 0" rpy="0 0 0" />
     </link>
-    <joint name="joint2_link2_joint" type="fixed">
+    <joint name="joint2_link3_joint" type="fixed">
         <parent link="joint2_link"/>
-        <child link="link2"/>
-        <origin xyz="0 ${link2_length/2} 0" rpy="${-pi/2} 0 0 "/>
+        <child link="link3"/>
+        <origin xyz="0 0 0" rpy="${-pi/2} 0 0 "/>
         <axis xyz="0 1 0"/>
     </joint>
-    <link name="link2">
+    <link name="link3">
             <visual>
                 <geometry>
-                    <cylinder radius="${link_radius}" length="${link2_length}"/>
+                    <cylinder radius="${link_radius}" length="${link_length}"/>
                 </geometry>
                 <material name="blue"/>
+                <origin xyz="0 0 ${link_length/2}" rpy="0 0 0 "/>
             </visual>
             <collision>
                 <geometry>
-                    <cylinder radius="${link_radius}" length="${link2_length}"/>
+                    <cylinder radius="${link_radius}" length="${link_length}"/>
                 </geometry>
             </collision>
-            <xacro:cylinder_inertia m="0.1" r="${link_radius}" h="${link2_length}"
+            <xacro:cylinder_inertia m="0.1" r="${link_radius}" h="${link_length}"
                                     xyz="0 0 0" rpy="0 0 0" />
     </link>
-    <joint name="link2_joint3" type="revolute">
-        <parent link="link2"/>
+    <joint name="link3_joint3" type="revolute">
+        <parent link="link3"/>
         <child link="joint3_link"/>
-        <origin xyz="0 0 ${link2_length/2}" rpy="${pi/2} 0 0"/>
+        <origin xyz="0 0 ${link_length}" rpy="${pi/2} 0 0"/>
         <limit effort="100.0" velocity="10.0" lower="${-pi/2}" upper="${pi/2}" />
         <axis xyz="0 0 1"/>
@@ -117,5 +107,5 @@
             <visual>
                 <geometry>
-                    <cylinder radius="${link_radius}" length="${joint_length}"/>
+                    <cylinder radius="${link_radius}" length="${link_length}"/>
                 </geometry>
                 <material name="black"/>
@@ -123,35 +113,36 @@
             <collision>
                 <geometry>
-                    <cylinder radius="${link_radius}" length="${joint_length}"/>
+                    <cylinder radius="${link_radius}" length="${link_length}"/>
                 </geometry>
             </collision>
-            <xacro:cylinder_inertia m="0.1" r="${link_radius}" h="${joint_length}"
+            <xacro:cylinder_inertia m="0.1" r="${link_radius}" h="${link_length}"
                                     xyz="0 0 0" rpy="0 0 0" />
     </link>
-    <joint name="joint3_link3_joint" type="fixed">
+    <joint name="joint3_link4_joint" type="fixed">
         <parent link="joint3_link"/>
-        <child link="link3"/>
-        <origin xyz="0 ${link3_length/2} 0" rpy="${-pi/2} 0 0 "/>
+        <child link="link4"/>
+        <origin xyz="0 0 0" rpy="${-pi/2} 0 0 "/>
         <axis xyz="0 1 0"/>
     </joint>
-    <link name="link3">
+    <link name="link4">
             <visual>
                 <geometry>
-                    <cylinder radius="${link_radius}" length="${link3_length}"/>
+                    <cylinder radius="${link_radius}" length="${link_length}"/>
                 </geometry>
                 <material name="blue"/>
+                <origin xyz="0 0 ${link_length/2}" rpy="0 0 0 "/>
             </visual>
             <collision>
                 <geometry>
-                    <cylinder radius="${link_radius}" length="${link3_length}"/>
+                    <cylinder radius="${link_radius}" length="${link_length}"/>
                 </geometry>
             </collision>
-            <xacro:cylinder_inertia m="0.1" r="${link_radius}" h="${link3_length}"
+            <xacro:cylinder_inertia m="0.1" r="${link_radius}" h="${link_length}"
                                     xyz="0 0 0" rpy="0 0 0" />
     </link>
-    <joint name="link3_payload" type="fixed">
-        <parent link="link3"/>
+    <joint name="link4_payload" type="fixed">
+        <parent link="link4"/>
         <child link="payload"/>
-        <origin xyz="0 0 ${link3_length/2 + payload_radius}" rpy="0 0 0"/>
+        <origin xyz="0 0 ${link_length + payload_radius}" rpy="0 0 0"/>
         <axis xyz="0 0 1"/>
     </joint>
@@ -162,4 +153,5 @@
             </geometry>
             <material name="grey"/>
+            <origin xyz="0 0 0" rpy="0 0 0 "/>
         </visual>
         <collision>
@@ -171,8 +163,3 @@
                                     xyz="0 0 0" rpy="0 0 0" />
     </link>
-    <gazebo>
-        <plugin filename="libgazebo_ros2_control.so" name="gazebo_ros2_control">
-            <parameters>$(find arm_robot_description)/config/3r_manipulator_control.yaml</parameters>
-        </plugin>
-    </gazebo>
 </robot>

File: src/arm_robot_description/urdf/common_properties.xacro (robot description, xacro)
@@ -1,32 +1,24 @@
 <?xml version="1.0"?>
 <robot xmlns:xacro="http://www.ros.org/wiki/xacro">
-    <material name="blue">
-        <color rgba="0 0 0.5 1" />
-    </material>
     <gazebo reference="base_link">
+        <material>Gazebo/Black</material>
+    </gazebo>
+    <gazebo reference="link1">
         <material>Gazebo/Blue</material>
     </gazebo>
-    <material name="grey">
-        <color rgba="0.5 0.5 0.5 1" />
-    </material>
-    <gazebo reference="base_link">
+    <gazebo reference="joint2_link">
+        <material>Gazebo/Black</material>
+    </gazebo>
+    <gazebo reference="link2">
         <material>Gazebo/Blue</material>
     </gazebo>
-    <gazebo reference="front_left_wheel">
+    <gazebo reference="joint3_link">
         <material>Gazebo/Black</material>
     </gazebo>
-    <gazebo reference="front_right_wheel">
-        <material>Gazebo/Black</material>
+    <gazebo reference="link3">
+        <material>Gazebo/Blue</material>
     </gazebo>
-    <gazebo reference="rear_left_wheel">
-        <material>Gazebo/Black</material>
-    </gazebo>
-    <gazebo reference="rear_right_wheel">
-        <material>Gazebo/Black</material>
-    </gazebo>
-    <gazebo reference="caster_wheel_link">
-        <material>Gazebo/Black</material>
-        <mul1 value="0.001" />
-        <mul2 value="0.001" />
+    <gazebo reference="payload">
+        <material>Gazebo/Grey</material>
     </gazebo>
     <xacro:macro name="box_inertia" params="m l w h xyz rpy">
