Commit message: Update arm_description.urdf.xacro

File: src/arm_robot_description/urdf/arm_description.urdf.xacro (robot description, xacro)
@@ -7,10 +7,10 @@
     <xacro:property name="link1_length" value="0.10" />
     <xacro:property name="link2_length" value="0.05" />
-    <xacro:property name="link3_length" value="0.04" />
+    <xacro:property name="link3_length" value="0.05" />
     <xacro:property name="payload_radius" value="0.0125" />
     <!-- Base footprint and link -->
     <link name="base_footprint">
         <inertial>
-            <mass value="0.001"/>
+            <mass value="1000"/>
             <inertia ixx="0.001" ixy="0.0" ixz="0.0" iyy="0.001" iyz="0.0" izz="0.001"/>
         </inertial>
@@ -25,5 +25,5 @@
         <child link="base_link"/>
         <origin xyz="0 0 ${link_radius}" rpy="${pi/2} 0 0"/>
-        <limit effort="100.0" velocity="10.0" lower="${-pi/2}" upper="${pi/2}" />
+        <limit effort="100.0" velocity="10.0" lower="0" upper="${pi}" />
         <axis xyz="0 0 1"/>
     </joint>
@@ -46,5 +46,5 @@
         <parent link="base_link"/>
         <child link="link1"/>
-        <origin xyz="0 ${link1_length/2} 0" rpy="${-pi/2} 0 0 "/>
+        <origin xyz="0 0 0" rpy="0 0 0 "/>
         <axis xyz="0 1 0"/>
     </joint>
@@ -55,4 +55,5 @@
                 </geometry>
                 <material name="blue"/>
+                <origin xyz="${link1_length/2} 0 0" rpy="0 ${pi/2} 0"/>
             </visual>
             <collision>
@@ -67,5 +68,5 @@
         <parent link="link1"/>
         <child link="joint2_link"/>
-        <origin xyz="0 0 ${link1_length/2}" rpy="${pi/2} 0 0"/>
+        <origin xyz="${link1_length} 0 0" rpy="0 0 0"/>
         <limit effort="100.0" velocity="10.0" lower="${-pi/2}" upper="${pi/2}" />
         <axis xyz="0 0 1"/>
@@ -89,5 +90,5 @@
         <parent link="joint2_link"/>
         <child link="link2"/>
-        <origin xyz="0 ${link2_length/2} 0" rpy="${-pi/2} 0 0 "/>
+        <origin xyz="0 0 0" rpy="0 0 0 "/>
         <axis xyz="0 1 0"/>
     </joint>
@@ -98,4 +99,5 @@
                 </geometry>
                 <material name="blue"/>
+                <origin xyz="${link2_length/2} 0 0" rpy="0 ${pi/2} 0"/>
             </visual>
             <collision>
@@ -110,5 +112,5 @@
         <parent link="link2"/>
         <child link="joint3_link"/>
-        <origin xyz="0 0 ${link2_length/2}" rpy="${pi/2} 0 0"/>
+        <origin xyz="${link2_length} 0 0" rpy="0 0 0"/>
         <limit effort="100.0" velocity="10.0" lower="${-pi/2}" upper="${pi/2}" />
         <axis xyz="0 0 1"/>
@@ -132,5 +134,5 @@
         <parent link="joint3_link"/>
         <child link="link3"/>
-        <origin xyz="0 ${link3_length/2} 0" rpy="${-pi/2} 0 0 "/>
+        <origin xyz="0 0 0" rpy="0 0 0 "/>
         <axis xyz="0 1 0"/>
     </joint>
@@ -141,4 +143,5 @@
                 </geometry>
                 <material name="blue"/>
+                <origin xyz="${link3_length/2} 0 0" rpy="0 ${pi/2} 0"/>
             </visual>
             <collision>
@@ -153,5 +156,5 @@
         <parent link="link3"/>
         <child link="payload"/>
-        <origin xyz="0 0 ${link3_length/2 + payload_radius}" rpy="0 0 0"/>
+        <origin xyz="${link3_length+ payload_radius} 0 0" rpy="0 0 0"/>
         <axis xyz="0 0 1"/>
     </joint>
